File: Amplifier TDA2030/TDA2030.kicad_pcb (KiCad board)
At the start: 2 copper layers, 61 x 34 mm, 27 parts, among them U1 TDA2030, X1 IN, X2 OUT, X3 PWR

Commit message: 20260719
Other:
- board text added: "260609"
- board text removed: "20260609"
Changed lines of the file:
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@@
   (gr_line (start 83.5 80) (end 113 80) (layer "Edge.Cuts") (width 0.1))
   (gr_arc (start 80 83.5) (mid 81.025126 81.025126) (end 83.5 80) (layer "Edge.Cuts") (width 0.1))
-  (gr_text "20260609" (at 94 82.5) (layer "B.Cu")
-    (effects (font (size 1.5 1.5) (thickness 0.15)) (justify mirror))
+  (gr_text "260609" (at 94 82.5) (layer "B.Cu")
+    (effects (font (size 2 2) (thickness 0.3)) (justify mirror))
   )
   (gr_text "GND" (at 105.5 109.5) (layer "F.SilkS")
@@
   )
   (gr_text "TDA20X0" (at 94 82.5) (layer "F.SilkS")
-    (effects (font (size 2 2) (thickness 0.2)))
+    (effects (font (size 2 2) (thickness 0.3)))
   )
   (gr_text "GND" (at 89.25 86.5) (layer "F.SilkS")
