File: Amplifier TDA2050 BTL/TDA2050.kicad_sch (KiCad schematic)
At the start: 30 parts, among them J1 IN, J2 OUT, U1 TDA2050, U2 TDA2050, X1 PWR

Commit message: 20260706
Other:
- title: (none) -> TDA2050 BTL Amplifier
Changed lines of the file:
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@@
 (kicad_sch (version 20211123) (generator eeschema)
   (paper "A4")
+  (title_block
+    (title "TDA2050 BTL Amplifier")
+  )
   (junction (at 34.29 172.72) (diameter 0) (color 0 0 0 0)
   )
