File: Amplifier TDA2050 BTL/TDA2050.kicad_pcb (KiCad board)
At the start: 2 copper layers, 74 x 39 mm, 30 parts, among them J1 IN, J2 OUT, U1 TDA2050, U2 TDA2050, X1 PWR

Commit message: 20260719
Other:
- board text added: "260618"
- board text removed: "20260618"
Changed lines of the file:
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@@
   (gr_arc (start 192.5 82.5) (mid 191.181981 85.681981) (end 188 87) (layer "Edge.Cuts") (width 0.1))
   (gr_line (start 118.5 82.5) (end 118.5 52.5) (layer "Edge.Cuts") (width 0.1))
-  (gr_text "20260618" (at 136 82) (layer "B.Cu")
-    (effects (font (size 1.5 1.5) (thickness 0.2)) (justify mirror))
+  (gr_text "260618" (at 137 82) (layer "B.Cu")
+    (effects (font (size 2 2) (thickness 0.3)) (justify mirror))
   )
   (gr_text "VEE" (at 179.8 75.08) (layer "F.SilkS")
@@
     (effects (font (size 2 2) (thickness 0.2)) (justify left))
   )
-  (gr_text "TDA2050 BTL" (at 136 82) (layer "F.SilkS")
-    (effects (font (size 2 2) (thickness 0.2)))
+  (gr_text "TDA2050 BTL" (at 137 82) (layer "F.SilkS")
+    (effects (font (size 2 2) (thickness 0.3)))
   )
   (gr_text "GND" (at 179.8 79.04) (layer "F.SilkS")
