File: Firealarm/F1.kicad_pcb (KiCad board)
At the start: 2 copper layers, 58 x 36 mm, 19 parts, among them Q1 BC548, Q2 BC548, Q3 BC548, SW1 ., X1 BATT., X2 LS

Commit message: 20260711
Parts:
- Q1, Q2, Q3: footprint fp:T -> Package_TO_SOT_THT:TO-92_Inline_Wide
- R1, R2, R3, R4, R5, R6: footprint fp:R -> Resistor_THT:R_Axial_DIN0207_L6.3mm_D2.5mm_P10.16mm_Horizontal
- X1: footprint fp:BATT -> Connector_JST:JST_PH_B2B-PH-K_1x02_P2.00mm_Vertical
- X2: footprint fp:KK2 -> Connector_Molex:Molex_KK-254_AE-6410-02A_1x02_P2.54mm_Vertical
- moved R1 2.17 mm to (108.0, 102.7)
- moved R2 2.17 mm to (96.0, 102.7)
- moved R3 2.17 mm to (102.0, 102.7)
- moved R4 2.17 mm to (114.0, 102.7)
- moved R5 2.17 mm to (120.0, 102.7)
- moved R6 2.17 mm to (126.0, 102.7)
- moved SW1 0.75 mm to (85.8, 111.0)
Routing:
- net Net-(C3-Pad1): track 29.1 -> 27.8 mm
- net Net-(R6-Pad1): track 8.86 -> 7.97 mm
- net VCC: track 42.8 -> 41.9 mm
- net GND: track 37.6 -> 36.7 mm
- net Net-(Q3-Pad1): track 3.54 -> 4.21 mm
- net Net-(C2-Pad1): track 16.4 -> 17.1 mm
- net Net-(C1-Pad1): track 17.5 -> 18.2 mm
- net Net-(C2-Pad2): track 27.6 -> 28.3 mm
- net Net-(R1-Pad2): track 25.6 -> 25.0 mm
- net Net-(C1-Pad2): track 10.7 -> 11.2 mm
Other:
- board text added: "260711"
