File: Firealarm/F1.kicad_sch (KiCad schematic)
At the start: 19 parts, among them Q1 BC548, Q2 BC548, Q3 BC548, SW1 ., X1 BATT., X2 LS

Commit message: 20260711
Parts:
- Q1, Q2, Q3: footprint fp:T -> Package_TO_SOT_THT:TO-92_Inline_Wide
- R1, R2, R3, R4, R5, R6: footprint fp:R -> Resistor_THT:R_Axial_DIN0207_L6.3mm_D2.5mm_P10.16mm_Horizontal
- X1: footprint fp:BATT -> Connector_JST:JST_PH_B2B-PH-K_1x02_P2.00mm_Vertical
- X2: footprint fp:KK2 -> Connector_Molex:Molex_KK-254_AE-6410-02A_1x02_P2.54mm_Vertical
Other:
- title: (none) -> Firealarm Tone Generator
Changed lines of the file:
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@@
 (kicad_sch (version 20211123) (generator eeschema)
   (paper "A4")
+  (title_block
+    (title "Firealarm Tone Generator")
+    (date "2026-07-11")
+  )
   (junction (at 83.82 96.52) (diameter 0) (color 0 0 0 0)
   )
@@
     (property "Reference" "R1" (id 0) (at 91.44 74.93 90))
     (property "Value" "220k" (id 1) (at 91.44 77.47 90))
-    (property "Footprint" "fp:R" (id 2) (at 91.44 79.502 90)
+    (property "Footprint" "Resistor_THT:R_Axial_DIN0207_L6.3mm_D2.5mm_P10.16mm_Horizontal" (id 2) (at 91.44 79.502 90)
       (effects (font (size 1.27 1.27)) hide)
     )
@@
       (effects (font (size 1.27 1.27)) (justify left))
     )
-    (property "Footprint" "fp:T" (id 2) (at 100.33 106.045 0)
+    (property "Footprint" "Package_TO_SOT_THT:TO-92_Inline_Wide" (id 2) (at 100.33 106.045 0)
       (effects (font (size 1.27 1.27) italic) (justify left) hide)
     )
@@
       (effects (font (size 1.27 1.27)) (justify left))
     )
-    (property "Footprint" "fp:R" (id 2) (at 131.572 87.63 90)
+    (property "Footprint" "Resistor_THT:R_Axial_DIN0207_L6.3mm_D2.5mm_P10.16mm_Horizontal" (id 2) (at 131.572 87.63 90)
       (effects (font (size 1.27 1.27)) hide)
     )
@@
       (effects (font (size 1.27 1.27)) (justify left))
     )
-    (property "Footprint" "fp:T" (id 2) (at 135.89 106.045 0)
+    (property "Footprint" "Package_TO_SOT_THT:TO-92_Inline_Wide" (id 2) (at 135.89 106.045 0)
       (effects (font (size 1.27 1.27) italic) (justify left) hide)
     )
@@
       (effects (font (size 1.27 1.27)) (justify right))
     )
-    (property "Footprint" "fp:R" (id 2) (at 117.348 87.63 90)
+    (property "Footprint" "Resistor_THT:R_Axial_DIN0207_L6.3mm_D2.5mm_P10.16mm_Horizontal" (id 2) (at 117.348 87.63 90)
       (effects (font (size 1.27 1.27)) hide)
     )
@@
       (effects (font (size 1.27 1.27)) (justify right))
     )
-    (property "Footprint" "fp:R" (id 2) (at 101.092 87.63 90)
+    (property "Footprint" "Resistor_THT:R_Axial_DIN0207_L6.3mm_D2.5mm_P10.16mm_Horizontal" (id 2) (at 101.092 87.63 90)
       (effects (font (size 1.27 1.27)) hide)
     )
@@
       (effects (font (size 1.27 1.27)) (justify left))
     )
-    (property "Footprint" "fp:T" (id 2) (at 156.21 106.045 0)
+    (property "Footprint" "Package_TO_SOT_THT:TO-92_Inline_Wide" (id 2) (at 156.21 106.045 0)
       (effects (font (size 1.27 1.27) italic) (justify left) hide)
     )
@@
       (effects (font (size 1.27 1.27)) (justify right))
     )
-    (property "Footprint" "fp:R" (id 2) (at 155.448 92.71 90)
+    (property "Footprint" "Resistor_THT:R_Axial_DIN0207_L6.3mm_D2.5mm_P10.16mm_Horizontal" (id 2) (at 155.448 92.71 90)
       (effects (font (size 1.27 1.27)) hide)
     )
@@
       (effects (font (size 1.27 1.27)) (justify right))
     )
-    (property "Footprint" "fp:BATT" (id 2) (at 182.88 107.95 0)
+    (property "Footprint" "Connector_JST:JST_PH_B2B-PH-K_1x02_P2.00mm_Vertical" (id 2) (at 182.88 107.95 0)
       (effects (font (size 1.27 1.27)) hide)
     )
@@
       (effects (font (size 1.27 1.27)) (justify right))
     )
-    (property "Footprint" "fp:KK2" (id 2) (at 161.29 83.82 0)
+    (property "Footprint" "Connector_Molex:Molex_KK-254_AE-6410-02A_1x02_P2.54mm_Vertical" (id 2) (at 161.29 83.82 0)
       (effects (font (size 1.27 1.27)) hide)
     )
@@
     (property "Reference" "R2" (id 0) (at 91.44 90.17 90))
     (property "Value" "100k" (id 1) (at 91.44 92.71 90))
-    (property "Footprint" "fp:R" (id 2) (at 91.44 98.298 90)
+    (property "Footprint" "Resistor_THT:R_Axial_DIN0207_L6.3mm_D2.5mm_P10.16mm_Horizontal" (id 2) (at 91.44 98.298 90)
       (effects (font (size 1.27 1.27)) hide)
     )
@@
     )
     (path "/0782bd35-2820-411c-9413-c35f7e3fbf9e"
-      (reference "Q1") (unit 1) (value "BC548") (footprint "fp:T")
+      (reference "Q1") (unit 1) (value "BC548") (footprint "Package_TO_SOT_THT:TO-92_Inline_Wide")
     )
     (path "/649a5dae-2589-4a13-a918-517625a4b87d"
-      (reference "Q2") (unit 1) (value "BC548") (footprint "fp:T")
+      (reference "Q2") (unit 1) (value "BC548") (footprint "Package_TO_SOT_THT:TO-92_Inline_Wide")
     )
     (path "/ab0b1e43-812c-470a-b096-2e95ab86418a"
-      (reference "Q3") (unit 1) (value "BC548") (footprint "fp:T")
+      (reference "Q3") (unit 1) (value "BC548") (footprint "Package_TO_SOT_THT:TO-92_Inline_Wide")
     )
     (path "/0179b30e-128b-4979-a2f9-92d626f718cc"
-      (reference "R1") (unit 1) (value "220k") (footprint "fp:R")
+      (reference "R1") (unit 1) (value "220k") (footprint "Resistor_THT:R_Axial_DIN0207_L6.3mm_D2.5mm_P10.16mm_Horizontal")
     )
     (path "/e968df06-081c-4395-b051-37b48b62c79b"
-      (reference "R2") (unit 1) (value "100k") (footprint "fp:R")
+      (reference "R2") (unit 1) (value "100k") (footprint "Resistor_THT:R_Axial_DIN0207_L6.3mm_D2.5mm_P10.16mm_Horizontal")
     )
     (path "/8b4ee033-504b-46ba-955a-b0e0ef81aba4"
-      (reference "R3") (unit 1) (value "4k7") (footprint "fp:R")
+      (reference "R3") (unit 1) (value "4k7") (footprint "Resistor_THT:R_Axial_DIN0207_L6.3mm_D2.5mm_P10.16mm_Horizontal")
     )
     (path "/7b3fa7fc-7ac7-4cf7-87b5-9f0815160543"
-      (reference "R4") (unit 1) (value "47k") (footprint "fp:R")
+      (reference "R4") (unit 1) (value "47k") (footprint "Resistor_THT:R_Axial_DIN0207_L6.3mm_D2.5mm_P10.16mm_Horizontal")
     )
     (path "/1019f9f4-bbe3-4c04-aa5e-97032f50dcdd"
-      (reference "R5") (unit 1) (value "4k7") (footprint "fp:R")
+      (reference "R5") (unit 1) (value "4k7") (footprint "Resistor_THT:R_Axial_DIN0207_L6.3mm_D2.5mm_P10.16mm_Horizontal")
     )
     (path "/b31c61e7-74df-4e89-8697-3d321c7d6ada"
-      (reference "R6") (unit 1) (value "220") (footprint "fp:R")
+      (reference "R6") (unit 1) (value "220") (footprint "Resistor_THT:R_Axial_DIN0207_L6.3mm_D2.5mm_P10.16mm_Horizontal")
     )
     (path "/0466051c-20cb-49c4-ab50-1a652205d7d3"
@@
     )
     (path "/c9422e5c-dadd-464b-936e-f5b2683355a9"
-      (reference "X1") (unit 1) (value "BATT.") (footprint "fp:BATT")
+      (reference "X1") (unit 1) (value "BATT.") (footprint "Connector_JST:JST_PH_B2B-PH-K_1x02_P2.00mm_Vertical")
     )
     (path "/d84d47c8-1416-456f-b2c5-52434240bcef"
-      (reference "X2") (unit 1) (value "LS") (footprint "fp:KK2")
-    )
-  )
+      (reference "X2") (unit 1) (value "LS") (footprint "Connector_Molex:Molex_KK-254_AE-6410-02A_1x02_P2.54mm_Vertical")
+    )
+  )
