File: LED Sound Power Meter/F2.kicad_pcb (KiCad board)
At the start: 2 copper layers, 100 x 35 mm, 36 parts, among them U1 LM386, U2 LM3914N, X1 BATT

Commit message: 20260719
Parts:
- added R4: 2k7, Resistor_THT:R_Axial_DIN0309_L9.0mm_D3.2mm_P12.70mm_Horizontal, F.Cu at (172.5, 88.5)
- moved R5 4.00 mm to (172.5, 92.5)
- moved R6 3.00 mm to (172.5, 96.5)
- moved R2 2.00 mm to (172.5, 100.5)
- moved R3 1.00 mm to (172.5, 104.5)
- renumbered R4 to R5, R5 to R6, R6 to R7, R7 to R8
Routing:
- net Net-(R6-Pad1): track 9.54 -> 26.3 mm
- net GND: track 186.3 -> 182.5 mm
- net Net-(R5-Pad1): track 16.7 -> 19.0 mm
- net Net-(JP1-Pad2): track 28.0 -> 26.8 mm
- net Net-(C6-Pad1): track 21.5 -> 20.7 mm
Other:
- board text added: "260717"
- board text removed: "260704"
