File: LED Sound Power Meter/F2.kicad_sch (KiCad schematic)
At the start: 36 parts, among them U1 LM386, U2 LM3914N, X1 BATT

Commit message: 20260719
Parts:
- added R4: 2k7, Resistor_THT:R_Axial_DIN0309_L9.0mm_D3.2mm_P12.70mm_Horizontal, symbol Device:R
- renumbered R4 to R5, R5 to R6, R6 to R7, R7 to R8
Connections:
- net at R5.1, U2.6 (RHI), U2.7 (REFOUT): now also R4.1
- net at R6.1, U2.8 (REFADJ): now also R4.2
Other:
- moved on the sheet: JP1, R5, R6

Commit message: 20260720
Parts:
- R4: now left out of the parts list
Changed lines of the file:
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@@
   )
   (symbol (lib_id "Device:R") (at 134.62 106.68 90) (mirror x) (unit 1)
-    (in_bom yes) (on_board yes) (fields_autoplaced)
+    (in_bom no) (on_board yes) (fields_autoplaced)
     (property "Reference" "R4" (id 0) (at 134.62 100.33 90))
     (property "Value" "2k7" (id 1) (at 134.62 102.87 90))
